File: HARDWARE/PCB/PCB_PAPI.kicad_pcb (KiCad board)
At the start: 6 copper layers, 23.4 x 26.8 mm, 64 parts, among them IC3 LDO40LPU33RY, IC5 LTC4065EDC#TRMPBF, IC6 MAX98357AETE+, J2 636101111001, J3 SM04B-GHS-TB_LF__SN_, J4 47309-2651, SW1 BOOTMODE, SW2 SW_Push, U5 ESP32-S3, Y2 LFXTAL069527REEL

Commit message: up
Parts:
- removed S1: 452404020202, samacsys2:452404020202
- removed U2: ~, Connector_JST:JST_SH_BM02B-SRSS-TB_1x02-1MP_P1.00mm_Vertical
- added C5: 100n, Capacitor_SMD:C_0201_0603Metric_Pad0.64x0.40mm_HandSolder, F.Cu at (158.3, 64.7)
- added G***: LOGO, LOGO, F.Cu at (158.4, 80.4)
- added J1: SM08B-GHS-TB__LF__SN_, samacsys2:SM08BGHSTBLFSN, B.Cu at (162.8, 63.5)
- added R2: 20k, Resistor_SMD:R_0201_0603Metric_Pad0.64x0.40mm_HandSolder, F.Cu at (159.7, 64.7)
- added R3: 20k, Resistor_SMD:R_0201_0603Metric_Pad0.64x0.40mm_HandSolder, F.Cu at (159.0, 64.7)
- moved R40 0.85 mm to (169.3, 75.6), turned to 0 degrees
- moved R29 0.62 mm to (163.5, 68.5)
- moved C4 0.57 mm to (175.7, 82.8)
- moved L5 0.30 mm to (173.7, 83.1)
- moved C3 0.21 mm to (171.8, 83.4)
- moved C67 0.13 mm to (166.2, 75.6)
- moved R4 0.12 mm to (167.0, 62.5)
Connections:
- J3 pad 5: (no net) -> GND
- J3 pad 6: (no net) -> GND
- U5 pad 19: unconnected-(U5-GPIO14-Pad19) -> /LED_TIM
- U5 pad 23: unconnected-(U5-GPIO17-Pad23) -> Net-(U5-GPIO17)
Routing:
- net GND: track 0.00 -> 25.4 mm, vias 0 -> 175
- net Net-(U5-GPIO17): track 0.00 -> 20.4 mm, vias 0 -> 2
- net /MAIN_BTN: track 1.01 -> 18.2 mm
- net /LED_TIM: track 0.00 -> 12.8 mm, vias 0 -> 1
- net +3.3V: track 7.55 -> 19.0 mm, vias 0 -> 25
- net /HP+: track 0.00 -> 11.3 mm, vias 0 -> 1
- net /HP-: track 0.00 -> 9.26 mm, vias 0 -> 1
- net Net-(C4-Pad1): track 0.00 -> 4.17 mm
- net Net-(C66-Pad1): track 0.00 -> 3.24 mm
- net VUSB: track 8.26 -> 10.9 mm, vias 0 -> 2
- net /LNA_IN: track 0.00 -> 2.39 mm
- net /D-: track 9.36 -> 7.43 mm
- net /D+: track 7.63 -> 6.13 mm
- net /SD_FSPICS: track 8.19 -> 9.04 mm
- net Net-(IC5-~{CHRG}): track 18.5 -> 17.6 mm
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- added copper zone on B.Cu, net +3.3V
- added copper zone on F.Cu, net +3.3V
- added copper zone on In2.Cu, net +3.3V
- added copper zone on B.Cu, net BAT+
- added copper zone on F.Cu, net BAT+
- added copper zone on B.Cu, net GND
- added copper zone on F.Cu, net GND
- added copper zone on In1.Cu, net GND
- added copper zone on In2.Cu, net GND
- added copper zone on F.Cu, net LDO_IN
- added copper zone on F.Cu, net Net-(C66-Pad1)
- added copper zone on F.Cu, net Net-(U5-VDD_SPI)
- added copper zone on B.Cu, net VUSB
Other:
- copper layers 6 -> 4
- board text added: "bat"
- board text added: "extension"
- board text added: "mathieu pommery"
- board text added: "usb"
