File: HARDWARE/PCB/PCB_PAPI.kicad_sch (KiCad schematic)
At the start: 64 parts, among them IC3 LDO40LPU33RY, IC5 LTC4065EDC#TRMPBF, IC6 MAX98357AETE+, J2 636101111001, J3 SM04B-GHS-TB_LF__SN_, J4 47309-2651, SW1 BOOTMODE, SW2 SW_Push, U5 ESP32-S3, Y2 LFXTAL069527REEL

Commit message: up
Parts:
- removed S1: 452404020202, samacsys2:452404020202, symbol samacsys2:452404020202
- removed U2: ~, Connector_JST:JST_SH_BM02B-SRSS-TB_1x02-1MP_P1.00mm_Vertical, symbol fc_h7:jst_2PIN
- added C5: 100n, Capacitor_SMD:C_0201_0603Metric_Pad0.64x0.40mm_HandSolder, symbol Device:C_Small
- added J1: SM08B-GHS-TB__LF__SN_, SM08BGHSTBLFSN, symbol samacsys2:SM08B-GHS-TB__LF__SN_
- added R2, R3: 20k, Resistor_SMD:R_0201_0603Metric_Pad0.64x0.40mm_HandSolder, symbol Device:R_Small
- J3: footprint samacsys:SM04B-GHS-TB -> SM04B-GHS-TB
Connections:
- net +3.3V: now also J1.4
- net BAT+: now also J1.3
- net GND: now also J3.5, J3.6, C5.2, J1.6, J1.MP1, J1.MP2, R3.2
- net HP+: now also J1.7
- net HP-: now also J1.8
- net LDO_IN: now also J1.2, R2.1
- net VUSB: now also J1.1
- net LED_TIM: now reaches U5.19 (GPIO14)
- net LED_TIM: now also J1.5
- net at U5.23 (GPIO17): now also C5.1, R2.2, R3.1
- no-connect marks 34 -> 32
Other:
- note added: "never use SPICS1,SPIHD,SPIWP,SPICS0,SPICLK,SPIQ,SPID,GPIO33,34,35,36,37"
- moved on the sheet: C1, C22, C24, C28, C29, C30, C44, C45, H1, H2, IC3, IC6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

Commit message: up
Other:
- note added: "CONNECTOR / MOUNTING HOLE"
- note added: "PERIPHERIAL"
- moved on the sheet: C1, C2, C22, C24, C28, C29, C3, C30, C4, C44, C45, H1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
